Commit message: Changed the colors of the arms

File: src/rebel_twin/urdf/rebel4dof_on_platform.gazebo.urdf.xacro (robot description, xacro)
@@ -14,10 +14,10 @@
     <origin xyz="0 0 0" rpy="0 0 0"/>
   </joint>
-  <gazebo reference="rebel_1_base_link"><gravity>0</gravity><material>Gazebo/DarkGrey</material></gazebo>
-  <gazebo reference="rebel_1_link_1"><gravity>0</gravity><material>Gazebo/DarkGrey</material></gazebo>
-  <gazebo reference="rebel_1_link_2"><gravity>0</gravity><material>Gazebo/FlatBlack</material></gazebo>
-  <gazebo reference="rebel_1_link_3"><gravity>0</gravity><material>Gazebo/DarkGrey</material></gazebo>
-  <gazebo reference="rebel_1_link_4"><gravity>0</gravity><material>Gazebo/DarkBlue</material></gazebo>
-  <gazebo reference="rebel_1_flange"><gravity>0</gravity><material>Gazebo/DarkGrey</material></gazebo>
+  <gazebo reference="rebel_1_base_link"><gravity>0</gravity><material>Gazebo/Grey</material></gazebo>
+  <gazebo reference="rebel_1_link_1"><gravity>0</gravity><material>Gazebo/Grey</material></gazebo>
+  <gazebo reference="rebel_1_link_2"><gravity>0</gravity><material>Gazebo/Grey</material></gazebo>
+  <gazebo reference="rebel_1_link_3"><gravity>0</gravity><material>Gazebo/Grey</material></gazebo>
+  <gazebo reference="rebel_1_link_4"><gravity>0</gravity><material>Gazebo/Grey</material></gazebo>
+  <gazebo reference="rebel_1_flange"><gravity>0</gravity><material>Gazebo/Grey</material></gazebo>
   <!-- Minimal ros2_control for the 4 arm joints, Gazebo backend -->
   <ros2_control name="rebel4dof_sim" type="system">

Commit message: rebel_twin: set link colours for twin visualisation

File: src/rebel_twin/urdf/rebel4dof_on_platform.gazebo.urdf.xacro (robot description, xacro)
@@ -14,10 +14,10 @@
     <origin xyz="0 0 0" rpy="0 0 0"/>
   </joint>
-  <gazebo reference="rebel_1_base_link"><gravity>0</gravity><material>Gazebo/Grey</material></gazebo>
-  <gazebo reference="rebel_1_link_1"><gravity>0</gravity><material>Gazebo/Grey</material></gazebo>
-  <gazebo reference="rebel_1_link_2"><gravity>0</gravity><material>Gazebo/Grey</material></gazebo>
-  <gazebo reference="rebel_1_link_3"><gravity>0</gravity><material>Gazebo/Grey</material></gazebo>
-  <gazebo reference="rebel_1_link_4"><gravity>0</gravity><material>Gazebo/Grey</material></gazebo>
-  <gazebo reference="rebel_1_flange"><gravity>0</gravity><material>Gazebo/Grey</material></gazebo>
+  <gazebo reference="rebel_1_base_link"><gravity>0</gravity><material>Gazebo/White</material></gazebo>
+  <gazebo reference="rebel_1_link_1"><gravity>0</gravity><material>Gazebo/White</material></gazebo>
+  <gazebo reference="rebel_1_link_2"><gravity>0</gravity><material>Gazebo/White</material></gazebo>
+  <gazebo reference="rebel_1_link_3"><gravity>0</gravity><material>Gazebo/White</material></gazebo>
+  <gazebo reference="rebel_1_link_4"><gravity>0</gravity><material>Gazebo/White</material></gazebo>
+  <gazebo reference="rebel_1_flange"><gravity>0</gravity><material>Gazebo/White</material></gazebo>
   <!-- Minimal ros2_control for the 4 arm joints, Gazebo backend -->
   <ros2_control name="rebel4dof_sim" type="system">

Commit message: Added a new world to the gazebo simulation and added a moveit configuration

File: src/rebel_twin/urdf/rebel4dof_on_platform.gazebo.urdf.xacro (robot description, xacro)
@@ -14,10 +14,10 @@
     <origin xyz="0 0 0" rpy="0 0 0"/>
   </joint>
-  <gazebo reference="rebel_1_base_link"><gravity>0</gravity><material>Gazebo/White</material></gazebo>
-  <gazebo reference="rebel_1_link_1"><gravity>0</gravity><material>Gazebo/White</material></gazebo>
-  <gazebo reference="rebel_1_link_2"><gravity>0</gravity><material>Gazebo/White</material></gazebo>
-  <gazebo reference="rebel_1_link_3"><gravity>0</gravity><material>Gazebo/White</material></gazebo>
-  <gazebo reference="rebel_1_link_4"><gravity>0</gravity><material>Gazebo/White</material></gazebo>
-  <gazebo reference="rebel_1_flange"><gravity>0</gravity><material>Gazebo/White</material></gazebo>
+  <gazebo reference="rebel_1_base_link"><material>Gazebo/Grey</material></gazebo>
+  <gazebo reference="rebel_1_link_1"><material>Gazebo/DarkGrey</material></gazebo>
+  <gazebo reference="rebel_1_link_2"><material>Gazebo/Grey</material></gazebo>
+  <gazebo reference="rebel_1_link_3"><material>Gazebo/DarkGrey</material></gazebo>
+  <gazebo reference="rebel_1_link_4"><material>Gazebo/Grey</material></gazebo>
+  <gazebo reference="rebel_1_flange"><material>Gazebo/DarkGrey</material></gazebo>
   <!-- Minimal ros2_control for the 4 arm joints, Gazebo backend -->
   <ros2_control name="rebel4dof_sim" type="system">
